Commit message: upload files

File: elaborato1/src/SCADA_Robot/urdf/scara_urdf_model.urdf (robot description, URDF)
Before this commit: robot myfirst, 9 links, 8 joints
Links:
- link L0: geometry visual box size=0.2 0.2 0.3
- link Li: geometry visual box size=0.2 0.2 0.3
Joints:
- joint joint_L0_to_M3: origin xyz=0.320 0.0 0.0 -> xyz=0.300 0.0 0.0
- joint joint_Li_to_M2: origin xyz=0.4 0.0 0.0 rpy=0.0 0.0 0.0 -> xyz=0.3 0.0 0.0 rpy=0.0 0.0 0.0
